Commit message: <Second Commit><update>更新limit的数据类型与ros2_controller

File: src/my_robot_moveit_config/config/my_robot.ros2_control.xacro (robot description, xacro)
@@ -2,5 +2,5 @@
 <robot xmlns:xacro="http://www.ros.org/wiki/xacro">
     <xacro:macro name="my_robot_ros2_control" params="name initial_positions_file">
-        <xacro:property name="initial_positions" value="${load_yaml(initial_positions_file)['initial_positions']}"/>
+        <xacro:property name="initial_positions" value="${xacro.load_yaml(initial_positions_file)['initial_positions']}"/>
         <ros2_control name="${name}" type="system">
             <hardware>
@@ -13,5 +13,4 @@
                   <param name="initial_value">${initial_positions['joint1']}</param>
                 </state_interface>
-                <state_interface name="velocity"/>
             </joint>
             <joint name="joint2">
@@ -20,5 +19,4 @@
                   <param name="initial_value">${initial_positions['joint2']}</param>
                 </state_interface>
-                <state_interface name="velocity"/>
             </joint>
             <joint name="joint3">
@@ -27,5 +25,4 @@
                   <param name="initial_value">${initial_positions['joint3']}</param>
                 </state_interface>
-                <state_interface name="velocity"/>
             </joint>
             <joint name="joint4">
@@ -34,5 +31,4 @@
                   <param name="initial_value">${initial_positions['joint4']}</param>
                 </state_interface>
-                <state_interface name="velocity"/>
             </joint>
             <joint name="joint5">
@@ -41,5 +37,4 @@
                   <param name="initial_value">${initial_positions['joint5']}</param>
                 </state_interface>
-                <state_interface name="velocity"/>
             </joint>
             <joint name="joint6">
@@ -48,5 +43,4 @@
                   <param name="initial_value">${initial_positions['joint6']}</param>
                 </state_interface>
-                <state_interface name="velocity"/>
             </joint>
         </ros2_control>
